File: PCB debug decoder/PC814/PC814.kicad_pcb (KiCad board)
At the start: 2 copper layers, 36.3 x 19.7 mm, 5 parts, among them P1 H1, P2 H2

Commit message: PCB decoder v0 update
Other:
- board outline removed
