File: PCB decoder/RFM95_shield_v0_1/RFM95_shield_v0_1.kicad_pcb (KiCad board)
At the start: 2 copper layers, 6 parts, among them J1 u.FL, J2 SMA, P1 H1, P2 H2, U1 RFM95

Commit message: Update 17/02/2021
Routing:
- net /GND: track 73.0 -> 38.1 mm
- added copper zone on F.Cu, net /GND
Changed lines of the file:
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@@
     (thickness 1.6)
     (drawings 0)
-    (tracks 63)
+    (tracks 57)
     (zones 0)
     (modules 6)
@@
   )
   (setup
-    (last_trace_width 0.45)
+    (last_trace_width 0.25)
     (user_trace_width 0.174244)
     (user_trace_width 0.45)
@@
     (trace_clearance 0.2)
     (zone_clearance 0.508)
-    (zone_45_only no)
+    (zone_45_only yes)
     (trace_min 0.2)
     (via_size 0.8)
@@
   (segment (start 122.8852 93.2434) (end 122.8852 93.2053) (width 0.174244) (layer F.Cu) (net 7))
   (segment (start 124.333 91.7956) (end 125.7808 93.2434) (width 0.174244) (layer F.Cu) (net 7))
-  (segment (start 124.334 101.299) (end 131.746 101.299) (width 0.68) (layer F.Cu) (net 7))
-  (segment (start 133.746 99.299) (end 140.334 99.299) (width 0.68) (layer F.Cu) (net 7))
-  (segment (start 131.746 101.299) (end 133.746 99.299) (width 0.68) (layer F.Cu) (net 7))
-  (segment (start 140.334 113.299) (end 135.905 113.299) (width 0.68) (layer F.Cu) (net 7))
-  (segment (start 131.746 109.14) (end 131.746 101.299) (width 0.68) (layer F.Cu) (net 7))
-  (segment (start 135.905 113.299) (end 131.746 109.14) (width 0.68) (layer F.Cu) (net 7))
   (segment (start 140.334 99.299) (end 140.334 98.299) (width 0.68) (layer F.Cu) (net 7))
   (segment (start 141.478 97.155) (end 143.383 97.155) (width 0.68) (layer F.Cu) (net 7))
@@
   (segment (start 140.334 107.299) (end 143.367 107.299) (width 0.68) (layer F.Cu) (net 13))
   (segment (start 124.334 94.7303) (end 124.334 99.299) (width 0.3429) (layer F.Cu) (net 14))
+  (zone (net 7) (net_name /GND) (layer F.Cu) (hatch edge 0.508)
+    (connect_pads (clearance 0.762))
+    (min_thickness 0.254)
+    (fill yes (arc_segments 32) (thermal_gap 0.508) (thermal_bridge_width 0.508))
+    (polygon
+      (pts
+        (xy 146.177 117.221) (xy 117.856 117.221) (xy 117.856 88.773) (xy 146.177 88.773)
+      )
+    )
+  )
+  (zone (net 0) (net_name "") (layer F.Cu) (hatch full 0.508)
+    (connect_pads (clearance 0.508))
+    (min_thickness 0.254)
+    (keepout (tracks not_allowed) (vias not_allowed) (copperpour not_allowed))
+    (fill (arc_segments 32) (thermal_gap 0.508) (thermal_bridge_width 0.508))
+    (polygon
+      (pts
+        (xy 139.319 113.792) (xy 125.349 113.792) (xy 125.349 98.806) (xy 139.319 98.806)
+      )
+    )
+  )
 )
